File: kicad/dotterboard/dotterboard.kicad_sch (KiCad schematic)
At the start: 5 parts, among them J1 Conn_01x04, J2 Conn_01x03, J3 Conn_01x03, SW1 SW_Push, U1 Pico

Commit message: Update schematic
Parts:
- added SW2: SW_Push, symbol Switch:SW_Push
Connections:
- net BTN_SET is gone; now on net BTN_UP: U1.9 (GPIO6)
- net GND: now also SW2.2
- net BTN_UP: now reaches SW1.1
- net BTN_CLR renamed BTN_DN
- net BTN_DN: now also SW2.1
Changed lines of the file:
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@@
 	(wire
 		(pts
+			(xy 106.68 144.78) (xy 105.41 144.78)
+		)
+		(stroke
+			(width 0)
+			(type default)
+		)
+	)
+	(wire
+		(pts
 			(xy 78.74 68.58) (xy 95.25 68.58)
 		)
@@
 	(wire
 		(pts
+			(xy 83.82 124.46) (xy 95.25 124.46)
+		)
+		(stroke
+			(width 0)
+			(type default)
+		)
+	)
+	(wire
+		(pts
 			(xy 195.0532 44.45) (xy 197.5932 44.45)
 		)
@@
 	(wire
 		(pts
+			(xy 83.82 144.78) (xy 95.25 144.78)
+		)
+		(stroke
+			(width 0)
+			(type default)
+		)
+	)
+	(wire
+		(pts
 			(xy 176.53 68.58) (xy 196.85 68.58)
 		)
@@
 	(wire
 		(pts
+			(xy 106.68 146.05) (xy 106.68 144.78)
+		)
+		(stroke
+			(width 0)
+			(type default)
+		)
+	)
+	(wire
+		(pts
 			(xy 191.77 97.79) (xy 196.85 97.79)
 		)
@@
 		)
 	)
-	(label "BTN_SET"
+	(label "BTN_UP"
 		(at 78.74 66.04 0)
 		(effects
@@
 		)
 	)
+	(label "BTN_UP"
+		(at 83.82 124.46 0)
+		(effects
+			(font
+				(size 1.27 1.27)
+			)
+			(justify left bottom)
+		)
+	)
 	(label "SLOT_SENSOR_I"
 		(at 78.74 83.82 0)
@@
 		)
 	)
+	(label "BTN_DN"
+		(at 83.82 144.78 0)
+		(effects
+			(font
+				(size 1.27 1.27)
+			)
+			(justify left bottom)
+		)
+	)
 	(label "OLED_I2C_SCL"
 		(at 179.07 100.33 0)
@@
 		)
 	)
-	(label "BTN_CLR"
+	(label "BTN_DN"
 		(at 78.74 68.58 0)
 		(effects
@@
 	(symbol
 		(lib_id "power:GND")
+		(at 106.68 146.05 0)
+		(unit 1)
+		(exclude_from_sim no)
+		(in_bom yes)
+		(on_board yes)
+		(dnp no)
+		(fields_autoplaced yes)
+		(property "Reference" "#PWR08"
+			(at 106.68 152.4 0)
+			(effects
+				(font
+					(size 1.27 1.27)
+				)
+				(hide yes)
+			)
+		)
+		(property "Value" "GND"
+			(at 106.68 151.13 0)
+			(effects
+				(font
+					(size 1.27 1.27)
+				)
+			)
+		)
+		(property "Footprint" ""
+			(at 106.68 146.05 0)
+			(effects
+				(font
+					(size 1.27 1.27)
+				)
+				(hide yes)
+			)
+		)
+		(property "Datasheet" ""
+			(at 106.68 146.05 0)
+			(effects
+				(font
+					(size 1.27 1.27)
+				)
+				(hide yes)
+			)
+		)
+		(property "Description" "Power symbol creates a global label with name \"GND\" , ground"
+			(at 106.68 146.05 0)
+			(effects
+				(font
+					(size 1.27 1.27)
+				)
+				(hide yes)
+			)
+		)
+		(pin "1"
+		)
+		(instances
+			(project "dotterboard"
+				(path "/5dba747f-0eb9-4b42-8c41-dd2ca3b3e1d8"
+					(reference "#PWR08")
+					(unit 1)
+				)
+			)
+		)
+	)
+	(symbol
+		(lib_id "power:GND")
 		(at 195.0532 49.53 0)
 		(unit 1)
@@
 					(unit 1)
 				)
+			)
+		)
+	)
+	(symbol
+		(lib_id "Switch:SW_Push")
+		(at 100.33 144.78 0)
+		(unit 1)
+		(exclude_from_sim no)
+		(in_bom yes)
+		(on_board yes)
+		(dnp no)
+		(fields_autoplaced yes)
+		(property "Reference" "SW2"
+			(at 100.33 137.16 0)
+			(effects
+				(font
+					(size 1.27 1.27)
+				)
+			)
+		)
+		(property "Value" "SW_Push"
+			(at 100.33 139.7 0)
+			(effects
+				(font
+					(size 1.27 1.27)
+				)
+			)
+		)
+		(property "Footprint" ""
+			(at 100.33 139.7 0)
+			(effects
+				(font
+					(size 1.27 1.27)
+				)
+				(hide yes)
+			)
+		)
+		(property "Datasheet" "~"
+			(at 100.33 139.7 0)
+			(effects
+				(font
+					(size 1.27 1.27)
+				)
+				(hide yes)
+			)
+		)
+		(property "Description" "Push button switch, generic, two pins"
+			(at 100.33 144.78 0)
+			(effects
+				(font
+					(size 1.27 1.27)
+				)
+				(hide yes)
+			)
+		)
+		(pin "1"
+		)
+		(pin "2"
+		)
+		(instances
+			(project "dotterboard"
+				(path "/5dba747f-0eb9-4b42-8c41-dd2ca3b3e1d8"
+					(reference "SW2")
+					(unit 1)
+				)
